Commit message: mobil taban modelinin oluşturuldu (collision ve inertia daha eklenmedi)

File: src/btkamr_description/urdf/mobile_base/main.urdf.xacro (robot description, xacro)
@@ -1,11 +1,12 @@
 <?xml version="1.0"?>
 <robot xmlns:xacro="http://www.ros.org/wiki/xacro" name="btkamr">
-<xacro:property name="chasis_l_x" value="0.6"/>
-<xacro:property name="chasis_l_y" value="0.4"/>
-<xacro:property name="chasis_l_z" value="0.2"/>
+<xacro:property name="chasis_len_x" value="0.6"/>
+<xacro:property name="chasis_len_y" value="0.4"/>
+<xacro:property name="chasis_len_z" value="0.2"/>
+<xacro:property name="base_chasis_offset" value="0.08"/>
 <xacro:include filename="./wheels.urdf.xacro"/>
 <link name="base_link"/>
 <joint name="base_TO_chasis" type="fixed">
-    <origin xyz="0.0 0.0 0.1" rpy="0.0 0.0 0.0"/>
+    <origin xyz="0.0 0.0 ${base_chasis_offset}" rpy="0.0 0.0 0.0"/>
     <parent link="base_link"/>
     <child link="chasis"/>
@@ -14,7 +15,13 @@
     <visual>
         <geometry>
-            <box size="${chasis_l_x} ${chasis_l_y} ${chasis_l_z}"/>
+            <box size="${chasis_len_x} ${chasis_len_y} ${chasis_len_z}"/>
         </geometry>
     </visual>
 </link>
+<link name="base_footprint"/>
+<joint name="base_TO_footprint" type="fixed">
+    <origin xyz="0.0 0.0 ${wh_radius}" rpy="0.0 0.0 0.0"/>
+    <parent link="base_footprint"/>
+    <child link="base_link"/>
+</joint>
 </robot>

File: src/btkamr_description/urdf/mobile_base/wheels.urdf.xacro (robot description, xacro)
@@ -3,33 +3,45 @@
     <xacro:property name="wh_thick" value="0.04"/>
     <xacro:property name="wh_chasis_gap" value="0.001"/>
-    <joint name="base_TO_wh_l" type="continuous">
-        <origin xyz="0.0 ${chasis_l_y / 2.0 + wh_thick + wh_chasis_gap} 0.0" rpy="0.0 0.0 0.0"/>
-        <parent link="base_link"/>
-        <child link="wh_l"/>
-        <axis xyz="0.0 1.0 0.0"/>
-        <limit lower="0.0" upper="0.0" effort="0.0" velocity="0.0"/>
-    </joint>
-    <link name="wh_l">
-        <visual>
-            <origin rpy="${pi / 2.0} 0.0 0.0"/>
-            <geometry>
-                <cylinder radius="${wh_radius}" length="${wh_thick}"/>
-            </geometry>
-        </visual>
-    </link>
-    <joint name="base_TO_wh_r" type="continuous">
-        <origin xyz="0.0 ${-1 * (chasis_l_y / 2.0 + wh_thick + wh_chasis_gap)} 0.0" rpy="0.0 0.0 0.0"/>
-        <parent link="base_link"/>
-        <child link="wh_r"/>
-        <axis xyz="0.0 1.0 0.0"/>
-        <limit lower="0.0" upper="0.0" effort="0.0" velocity="0.0"/>
-    </joint>
-    <link name="wh_r">
-        <visual>
-            <origin rpy="${pi / 2.0} 0.0 0.0"/>
-            <geometry>
-                <cylinder radius="${wh_radius}" length="${wh_thick}"/>
-            </geometry>
-        </visual>
-    </link>
+    <xacro:property name="cwh_radius" value="${(wh_radius - (chasis_len_z / 2.0 - base_chasis_offset)) / 2.0}"/>
+    <xacro:property name="cwh_chasis_offset" value="0.1"/>
+    <!-- Wheels -->
+    <xacro:macro name="create_wh" params="postfix yfact">
+        <joint name="base_TO_wh_${postfix}" type="continuous">
+            <origin xyz="0.0 ${yfact * (chasis_len_y / 2.0 + wh_thick + wh_chasis_gap)} 0.0" rpy="0.0 0.0 0.0"/>
+            <parent link="base_link"/>
+            <child link="wh_${postfix}"/>
+            <axis xyz="0.0 1.0 0.0"/>
+            <limit lower="0.0" upper="0.0" effort="0.0" velocity="0.0"/>
+        </joint>
+        <link name="wh_${postfix}">
+            <visual>
+                <origin rpy="${pi / 2.0} 0.0 0.0"/>
+                <geometry>
+                    <cylinder radius="${wh_radius}" length="${wh_thick}"/>
+                </geometry>
+            </visual>
+        </link>
+    </xacro:macro>
+    <xacro:create_wh postfix="l" yfact="1.0"/>
+    <xacro:create_wh postfix="r" yfact="-1.0"/>
+    <!-- Caster Wheels -->
+    <xacro:macro name="create_cwh" params="postfix xfact yfact">
+        <joint name="chasis_TO_cwh_${postfix}" type="continuous">
+            <origin xyz="${xfact * (chasis_len_x / 2.0 - cwh_chasis_offset)} ${yfact * (chasis_len_y / 2.0 - cwh_chasis_offset)} ${-1 * (chasis_len_z / 2.0 + cwh_radius)}" rpy="0.0 0.0 0.0"/>
+            <parent link="chasis"/>
+            <child link="cwh_${postfix}"/>
+            <axis xyz="0.0 1.0 0.0"/>
+        </joint>
+        <link name="cwh_${postfix}">
+            <visual>
+                <geometry>
+                    <sphere radius="${cwh_radius}"/>
+                </geometry>
+            </visual>
+        </link>
+    </xacro:macro>
+    <xacro:create_cwh postfix="lf" xfact="1.0" yfact="1.0"/>
+    <xacro:create_cwh postfix="lb" xfact="-1.0" yfact="1.0"/>
+    <xacro:create_cwh postfix="rf" xfact="1.0" yfact="-1.0"/>
+    <xacro:create_cwh postfix="rb" xfact="-1.0" yfact="-1.0"/>
 </robot>

Commit message: renklendirme yapıldı.

File: src/btkamr_description/urdf/mobile_base/main.urdf.xacro (robot description, xacro)
@@ -5,4 +5,5 @@
 <xacro:property name="chasis_len_z" value="0.2"/>
 <xacro:property name="base_chasis_offset" value="0.08"/>
+<xacro:include filename="../common_props.xacro"/>
 <xacro:include filename="./wheels.urdf.xacro"/>
 <link name="base_link"/>
@@ -17,4 +18,5 @@
             <box size="${chasis_len_x} ${chasis_len_y} ${chasis_len_z}"/>
         </geometry>
+        <material name="green"/>
     </visual>
 </link>

File: src/btkamr_description/urdf/mobile_base/wheels.urdf.xacro (robot description, xacro)
@@ -20,4 +20,5 @@
                     <cylinder radius="${wh_radius}" length="${wh_thick}"/>
                 </geometry>
+                <material name="gray"/>
             </visual>
         </link>
@@ -38,4 +39,5 @@
                     <sphere radius="${cwh_radius}"/>
                 </geometry>
+                <material name="gray"/>
             </visual>
         </link>
