Commit message: basit geometri ile oluşturulacak linkler için macro tanımlandı (kolaylık olması için hazır inertia collision ve visual)

File: src/btkamr_description/urdf/common_props.xacro (robot description, xacro)
@@ -18,3 +18,89 @@
         <color rgba="0.6 0.6 0.6 1.0"/>
     </material>
+    <xacro:macro name="box_inertia" params="mass lenx leny lenz">
+        <mass value="${mass}"/>
+        <inertia
+            ixx="${mass * (leny*leny + lenz*lenz) / 12.0}"
+            iyy="${mass * (lenx*lenx + lenz*lenz) / 12.0}"
+            izz="${mass * (lenx*lenx + leny*leny) / 12.0}"
+            ixy="0" ixz="0" iyz="0"
+        />
+    </xacro:macro>
+    <xacro:macro name="cylinder_inertia" params="mass radius length">
+        <mass value="${mass}"/>
+        <inertia
+            ixx="${mass * (3*radius*radius + length*length) / 12.0}"
+            iyy="${mass * (3*radius*radius + length*length) / 12.0}"
+            izz="${mass * (radius*radius) / 2.0}"
+            ixy="0" ixz="0" iyz="0"
+        />
+    </xacro:macro>
+    <xacro:macro name="sphere_inertia" params="mass radius">
+        <mass value="${mass}"/>
+        <inertia
+            ixx="${2.0 * mass * radius * radius / 5.0}"
+            iyy="${2.0 * mass * radius * radius / 5.0}"
+            izz="${2.0 * mass * radius * radius / 5.0}"
+            ixy="0" ixz="0" iyz="0"
+        />
+    </xacro:macro>
+    <xacro:macro name="create_box_link" params="name oxyz orpy lenx leny lenz mass material">
+        <link name="${name}">
+            <inertial>
+                <origin xyz="${oxyz}" rpy="${orpy}"/>
+                <xacro:box_inertia mass="${mass}" lenx="${lenx}" leny="${leny}" lenz="${lenz}"/>
+            </inertial>
+            <visual>
+                <origin xyz="${oxyz}" rpy="${orpy}"/>
+                <geometry><box size="${lenx} ${leny} ${lenz}"/></geometry>
+                <material name="${material}"/>
+            </visual>
+            <collision>
+                <origin xyz="${oxyz}" rpy="${orpy}"/>
+                <geometry><box size="${lenx} ${leny} ${lenz}"/></geometry>
+            </collision>
+        </link>
+    </xacro:macro>
+    <xacro:macro name="create_cylinder_link" params="name oxyz orpy radius length mass material">
+        <link name="${name}">
+            <inertial>
+                <origin xyz="${oxyz}" rpy="${orpy}"/>
+                <xacro:cylinder_inertia mass="${mass}" radius="${radius}" length="${length}"/>
+            </inertial>
+            <visual>
+                <origin xyz="${oxyz}" rpy="${orpy}"/>
+                <geometry>
+                    <cylinder radius="${radius}" length="${length}"/>
+                </geometry>
+                <material name="${material}"/>
+            </visual>
+            <collision>
+                <origin xyz="${oxyz}" rpy="${orpy}"/>
+                <geometry>
+                    <cylinder radius="${radius}" length="${length}"/>
+                </geometry>
+            </collision>
+        </link>
+    </xacro:macro>
+    <xacro:macro name="create_sphere_link" params="name oxyz orpy radius mass material">
+        <link name="${name}">
+            <inertial>
+                <origin xyz="${oxyz}" rpy="${orpy}"/>
+                <xacro:sphere_inertia mass="${mass}" radius="${radius}"/>
+            </inertial>
+            <visual>
+                <origin xyz="${oxyz}" rpy="${orpy}"/>
+                <geometry>
+                    <sphere radius="${radius}"/>
+                </geometry>
+                <material name="${material}"/>
+            </visual>
+            <collision>
+                <origin xyz="${oxyz}" rpy="${orpy}"/>
+                <geometry>
+                    <sphere radius="${radius}"/>
+                </geometry>
+            </collision>
+        </link>
+    </xacro:macro>
 </robot>

File: src/btkamr_description/urdf/mobile_base/main.urdf.xacro (robot description, xacro)
@@ -5,4 +5,5 @@
 <xacro:property name="chasis_len_z" value="0.2"/>
 <xacro:property name="base_chasis_offset" value="0.08"/>
+<xacro:property name="chasis_mass" value="2.0"/>
 <xacro:include filename="../common_props.xacro"/>
 <xacro:include filename="./wheels.urdf.xacro"/>
@@ -13,12 +14,14 @@
     <child link="chasis"/>
 </joint>
-<link name="chasis">
-    <visual>
-        <geometry>
-            <box size="${chasis_len_x} ${chasis_len_y} ${chasis_len_z}"/>
-        </geometry>
-        <material name="green"/>
-    </visual>
-</link>
+<xacro:create_box_link
+    name="chasis"
+    oxyz="0.0 0.0 0.0"
+    orpy="0.0 0.0 0.0"
+    lenx="${chasis_len_x}"
+    leny="${chasis_len_y}"
+    lenz="${chasis_len_z}"
+    mass="${chasis_mass}"
+    material="green"
+/>
 <link name="base_footprint"/>
 <joint name="base_TO_footprint" type="fixed">

File: src/btkamr_description/urdf/mobile_base/wheels.urdf.xacro (robot description, xacro)
@@ -3,6 +3,8 @@
     <xacro:property name="wh_thick" value="0.04"/>
     <xacro:property name="wh_chasis_gap" value="0.001"/>
+    <xacro:property name="wh_mass" value="1.0"/>
     <xacro:property name="cwh_radius" value="${(wh_radius - (chasis_len_z / 2.0 - base_chasis_offset)) / 2.0}"/>
     <xacro:property name="cwh_chasis_offset" value="0.1"/>
+    <xacro:property name="cwh_mass" value="0.1"/>
     <!-- Wheels -->
     <xacro:macro name="create_wh" params="postfix yfact">
@@ -12,15 +14,14 @@
             <child link="wh_${postfix}"/>
             <axis xyz="0.0 1.0 0.0"/>
-            <limit lower="0.0" upper="0.0" effort="0.0" velocity="0.0"/>
         </joint>
-        <link name="wh_${postfix}">
-            <visual>
-                <origin rpy="${pi / 2.0} 0.0 0.0"/>
-                <geometry>
-                    <cylinder radius="${wh_radius}" length="${wh_thick}"/>
-                </geometry>
-                <material name="gray"/>
-            </visual>
-        </link>
+        <xacro:create_cylinder_link
+            name="wh_${postfix}"
+            oxyz="0.0 0.0 0.0"
+            orpy="${pi / 2.0} 0.0 0.0"
+            radius="${wh_radius}"
+            length="${wh_thick}"
+            mass="${wh_mass}"
+            material="gray"
+        />
     </xacro:macro>
     <xacro:create_wh postfix="l" yfact="1.0"/>
@@ -34,12 +35,12 @@
             <axis xyz="0.0 1.0 0.0"/>
         </joint>
-        <link name="cwh_${postfix}">
-            <visual>
-                <geometry>
-                    <sphere radius="${cwh_radius}"/>
-                </geometry>
-                <material name="gray"/>
-            </visual>
-        </link>
+        <xacro:create_sphere_link
+            name="cwh_${postfix}"
+            oxyz="0.0 0.0 0.0"
+            orpy="0.0 0.0 0.0"
+            radius="${cwh_radius}"
+            mass="${cwh_mass}"
+            material="gray"
+        />
     </xacro:macro>
     <xacro:create_cwh postfix="lf" xfact="1.0" yfact="1.0"/>
